File: ldo.kicad_sch (KiCad schematic)
At the start: 3 parts

Commit message: v1
Parts:
- gave numbers to parts that had none: 3
Changed lines of the file:
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@@
 		(dnp no)
 		(fields_autoplaced yes)
-		(property "Reference" "#PWR010"
+		(property "Reference" "#PWR022"
 			(at 134.62 114.3 0)
 			(effects
@@
 			(project "aroma"
 				(path "/41d97073-34b5-4be3-afd3-c3d0ba6d78a9/f4040f6c-cfda-4124-94c1-e2a6c2f7e4ba"
-					(reference "#PWR010")
+					(reference "#PWR022")
 					(unit 1)
 				)
@@
 		(dnp no)
 		(fields_autoplaced yes)
-		(property "Reference" "#PWR09"
+		(property "Reference" "#PWR021"
 			(at 129.54 90.17 0)
 			(effects
@@
 			(project "aroma"
 				(path "/41d97073-34b5-4be3-afd3-c3d0ba6d78a9/f4040f6c-cfda-4124-94c1-e2a6c2f7e4ba"
-					(reference "#PWR09")
+					(reference "#PWR021")
 					(unit 1)
 				)
@@
 		(dnp no)
 		(fields_autoplaced yes)
-		(property "Reference" "C?"
+		(property "Reference" "C13"
 			(at 167.64 99.0599 0)
 			(effects
@@
 			(project "aroma"
 				(path "/41d97073-34b5-4be3-afd3-c3d0ba6d78a9/f4040f6c-cfda-4124-94c1-e2a6c2f7e4ba"
-					(reference "C?")
+					(reference "C13")
 					(unit 1)
 				)
@@
 		(dnp no)
 		(fields_autoplaced yes)
-		(property "Reference" "#PWR012"
+		(property "Reference" "#PWR024"
 			(at 163.83 114.3 0)
 			(effects
@@
 			(project "aroma"
 				(path "/41d97073-34b5-4be3-afd3-c3d0ba6d78a9/f4040f6c-cfda-4124-94c1-e2a6c2f7e4ba"
-					(reference "#PWR012")
+					(reference "#PWR024")
 					(unit 1)
 				)
@@
 		(dnp no)
 		(fields_autoplaced yes)
-		(property "Reference" "C?"
+		(property "Reference" "C12"
 			(at 138.43 99.0599 0)
 			(effects
@@
 			(project "aroma"
 				(path "/41d97073-34b5-4be3-afd3-c3d0ba6d78a9/f4040f6c-cfda-4124-94c1-e2a6c2f7e4ba"
-					(reference "C?")
+					(reference "C12")
 					(unit 1)
 				)
@@
 		(dnp no)
 		(fields_autoplaced yes)
-		(property "Reference" "#PWR015"
+		(property "Reference" "#PWR025"
 			(at 168.91 90.17 0)
 			(effects
@@
 			(project "aroma"
 				(path "/41d97073-34b5-4be3-afd3-c3d0ba6d78a9/f4040f6c-cfda-4124-94c1-e2a6c2f7e4ba"
-					(reference "#PWR015")
+					(reference "#PWR025")
 					(unit 1)
 				)
@@
 		(dnp no)
 		(fields_autoplaced yes)
-		(property "Reference" "U?"
+		(property "Reference" "U2"
 			(at 149.86 87.63 0)
 			(effects
@@
 			(project "aroma"
 				(path "/41d97073-34b5-4be3-afd3-c3d0ba6d78a9/f4040f6c-cfda-4124-94c1-e2a6c2f7e4ba"
-					(reference "U?")
+					(reference "U2")
 					(unit 1)
 				)
@@
 		(dnp no)
 		(fields_autoplaced yes)
-		(property "Reference" "#PWR011"
+		(property "Reference" "#PWR023"
 			(at 149.86 114.3 0)
 			(effects
@@
 			(project "aroma"
 				(path "/41d97073-34b5-4be3-afd3-c3d0ba6d78a9/f4040f6c-cfda-4124-94c1-e2a6c2f7e4ba"
-					(reference "#PWR011")
-					(unit 1)
-				)
+					(reference "#PWR023")
+					(unit 1)
+				)
