File: untitled.kicad_sch (KiCad schematic)
At the start: 1 part

Commit message: passed drc (somehow)
board routing is def cooked
verify:
- boost layout
- usb terminal layout
Parts:
- U5: renamed from U4; footprint (none) -> footprints:LCD_ST7789
Changed lines of the file:
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@@
 		(dnp no)
 		(fields_autoplaced yes)
-		(property "Reference" "#PWR045"
+		(property "Reference" "#PWR053"
 			(at 138.43 83.82 0)
 			(effects
@@
 			(project ""
 				(path "/41d97073-34b5-4be3-afd3-c3d0ba6d78a9/a9cd5c70-79f3-4074-a76f-afa3a3607378"
-					(reference "#PWR045")
+					(reference "#PWR053")
 					(unit 1)
 				)
@@
 		(dnp no)
 		(fields_autoplaced yes)
-		(property "Reference" "U4"
+		(property "Reference" "U5"
 			(at 166.37 98.4249 0)
 			(effects
@@
 			)
 		)
-		(property "Footprint" ""
+		(property "Footprint" "footprints:LCD_ST7789"
 			(at 158.75 81.28 0)
 			(effects
@@
 			(project ""
 				(path "/41d97073-34b5-4be3-afd3-c3d0ba6d78a9/a9cd5c70-79f3-4074-a76f-afa3a3607378"
-					(reference "U4")
+					(reference "U5")
 					(unit 1)
 				)
@@
 		(dnp no)
 		(fields_autoplaced yes)
-		(property "Reference" "#PWR046"
+		(property "Reference" "#PWR054"
 			(at 138.43 104.14 0)
 			(effects
@@
 			(project ""
 				(path "/41d97073-34b5-4be3-afd3-c3d0ba6d78a9/a9cd5c70-79f3-4074-a76f-afa3a3607378"
-					(reference "#PWR046")
+					(reference "#PWR054")
 					(unit 1)
 				)
