File: aroma.kicad_pcb (KiCad board)
At the start: 4 copper layers, 96 x 44 mm, 108 parts, among them IC1 ESP32-WROOM-32E-N8R2, J1 USB4105-GF-A, J2 691137710003, J3 691137710002, J4 691137710002, J5 691137710002, J6 691137710002, J7 691137710002, J8 691137710002, J9 691137710002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

Commit message: gerber fix
Parts:
- renumbered TP5 to 12V, TP3 to 3V3
Routing:
- net Net-(SW3-PUSH_(N.O.)): track 26.1 -> 24.9 mm
- net GND: vias 67 -> 66
- net /LCD Display/TCS: vias 4 -> 3
- net /LCD Display/RST: vias 4 -> 3
Changed lines of the file:
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@@
 		(layer "F.Cu")
 		(at 130 100.5 180)
-		(property "Reference" "TP5"
+		(property "Reference" "12V"
 			(at 0 1.8 180)
 			(layer "F.SilkS")
@@
 		(layer "F.Cu")
 		(at 198.5 112.2)
-		(property "Reference" "TP3"
+		(property "Reference" "3V3"
 			(at -2.8 0 0)
 			(layer "F.SilkS")
@@
 		(net 1)
 	)
-	(via
-		(at 144 104.25)
-		(size 0.6)
-		(drill 0.3)
-		(layers "F.Cu" "B.Cu")
-		(free yes)
-		(net 1)
-	)
 	(segment
 		(start 160.298098 100.55)
@@
 		(net 47)
 	)
-	(via
-		(at 151.1 85.5)
-		(size 0.6)
-		(drill 0.3)
-		(layers "F.Cu" "B.Cu")
-		(net 47)
-	)
 	(segment
 		(start 129.075 86.05)
@@
 	)
 	(via
-		(at 150.7 86.3)
-		(size 0.6)
-		(drill 0.3)
-		(layers "F.Cu" "B.Cu")
-		(net 51)
-	)
-	(via
 		(at 129.417215 86.808647)
 		(size 0.6)
@@
 		(width 0.2)
 		(layer "B.Cu")
-		(net 71)
-	)
-	(segment
-		(start 192.1 97.4)
-		(end 192.1 96.25)
-		(width 0.2)
-		(layer "B.Cu")
